File: zero-2w-radio.kicad_sch (KiCad schematic)
At the start: 5 parts, among them J1 Raspberry_Pi_2_3, U1 nRF52840_Dongle

Commit message: Updated some footprints
Parts:
- J1: footprint Connector_PinHeader_2.54mm:PinHeader_2x20_P2.54mm_Vertical -> Connector_PinHeader_2.54mm:PinHeader_2x05_P2.54mm_Vertical
- JP3: footprint Connector_PinHeader_2.54mm:PinHeader_1x02_P2.54mm_Horizontal -> Connector_PinHeader_2.54mm:PinHeader_1x02_P2.54mm_Vertical
Connections:
- net VDD: now also JP2.2 (B); no longer JP2.1 (A)
- net at JP1.1 (A), JP3.1 (A): now also JP2.1 (A); no longer JP2.2 (B)
Other:
- moved on the sheet: JP2
Changed lines of the file:
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@@
 			)
 		)
-		(property "Footprint" "Connector_PinHeader_2.54mm:PinHeader_2x20_P2.54mm_Vertical"
+		(property "Footprint" "Connector_PinHeader_2.54mm:PinHeader_2x05_P2.54mm_Vertical"
 			(at 59.69 67.31 0)
 			(effects
@@
 			)
 		)
-		(property "Footprint" "Connector_PinHeader_2.54mm:PinHeader_1x02_P2.54mm_Horizontal"
+		(property "Footprint" "Connector_PinHeader_2.54mm:PinHeader_1x02_P2.54mm_Vertical"
 			(at 218.44 55.88 0)
 			(effects
@@
 	(symbol
 		(lib_id "Jumper:SolderJumper_2_Open")
-		(at 218.44 45.72 0)
+		(at 218.44 45.72 180)
 		(unit 1)
 		(exclude_from_sim yes)
